File: pcb/tailplug/tailplug.kicad_sch (KiCad schematic)
At the start: 0 parts

Commit message: Add work from 2025-07-20
Parts:
- added J1: Conn_01x06, Connector_PinHeader_2.00mm:PinHeader_1x06_P2.00mm_Vertical, symbol Connector_Generic:Conn_01x06
- added UTP1: ~, Connector_PinHeader_2.54mm:PinHeader_1x08_P2.54mm_Vertical, symbol tailplug:Tailplug_Male
Connections:
- new net: UTP1.1 (CONT), UTP1.2 (CONT)
- new net: J1.1 (Pin_1), UTP1.3 (OUT)
- new net: J1.2 (Pin_2), UTP1.4 (GND)
- new net: J1.3 (Pin_3), UTP1.5 (UART_RX)
- new net: J1.4 (Pin_4), UTP1.6 (UART_TX)
- new net: J1.5 (Pin_5), UTP1.7 (5V_PWM)
- new net: J1.6 (Pin_6), UTP1.8 (24V_PWM)
