File: pcb/tailplug/tailplug.kicad_pcb (KiCad board)
At the start: 2 copper layers, 14.5 x 25 mm, 5 parts, among them J1 Conn_01x06

Commit message: Replace boykissers on PCBs with my pfp (copyright reasons :3)
Parts:
- added G***: LOGO, LOGO, F.Cu at (10.0, 21.2)
Other:
- board text added: "xt-1"
- board text removed: "xt-1 / redbigz.com"
